File: {{cookiecutter.project_name}}/{{cookiecutter.project_name}}.kicad_sch (KiCad schematic)
At the start: 3 parts

Commit message: Exclude tooling from BOM/CPL
Parts:
- H1, H2, H3: now left out of the parts list
Changed lines of the file:
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@@
 		(unit 1)
 		(exclude_from_sim no)
-		(in_bom yes)
+		(in_bom no)
 		(on_board yes)
 		(dnp no)
@@
 		(unit 1)
 		(exclude_from_sim no)
-		(in_bom yes)
+		(in_bom no)
 		(on_board yes)
 		(dnp no)
@@
 		(unit 1)
 		(exclude_from_sim no)
-		(in_bom yes)
+		(in_bom no)
 		(on_board yes)
 		(dnp no)
