File: {{cookiecutter.project_name}}/{{cookiecutter.project_name}}.kicad_pcb (KiCad board)
At the start: 2 copper layers, 0 parts

Commit message: Add basic PCB
Parts:
- added H1: ~, PCM_JLCPCB:Hole_Tooling_JLCPCB, F.Cu at (33.0, 33.0)
- added H2: ~, PCM_JLCPCB:Hole_Tooling_JLCPCB, F.Cu at (127.0, 33.0)
- added H3: ~, PCM_JLCPCB:Hole_Tooling_JLCPCB, F.Cu at (33.0, 127.0)
Other:
- board outline added: 100 x 100 mm
